File: FPSP Camera.kicad_sch (KiCad schematic)
At the start: 79 parts, among them J1 USB_B_Micro, J2 Conn_02x06_Odd_Even, J3 SM03B-SRSS-TB, J4 Conn_01x24_Socket, J5 Conn_02x04_Counter_Clockwise, J6 Conn_02x07_Counter_Clockwise, U1 TLV75533PDRV, U2 TLV73328PDRV, U3 RP2350_60QFN, U4 TLV73315PDRV, U5 W25Q128JVS, U6 ICM-45686, Y1 SiT8008xx-1x-xxE

Commit message: routing updates
Parts:
- removed C19: 100n, Capacitor_SMD:C_0402_1005Metric, symbol Device:C
- L1: footprint Inductor_SMD:L_1210_3225Metric -> Inductor_SMD:L_pol_2016
- renumbered C27 to C1, C16 to C10, C20 to C11, C21 to C12, C23 to C13, C24 to C14, C28 to C15, C30 to C16, C7 to C17, C2 to C18, C3 to C19, C29 to C2, C22 to C20, C31 to C21, C32 to C22, C26 to C23, C25 to C24, C18 to C25, C1 to C26, C5 to C27, C9 to C28, C10 to C29, C4 to C3, C13 to C30, C17 to C31, C6 to C4, C8 to C5, C11 to C6, C12 to C7, C14 to C8, C15 to C9, J4 to J1, J5 to J2, J6 to J3, J3 to J4, J1 to J5, J2 to J6, R16 to R1, R4 to R10, R13 to R11, R18 to R12, R14 to R13, R19 to R14, R3 to R15, R20 to R16, R22 to R17, R10 to R18, R11 to R19, R12 to R20, R15 to R21, R5 to R3, R6 to R4, R9 to R5, R1 to R6, R17 to R9, U6 to U1, U5 to U2, U1 to U4, U2 to U5, U4 to U6
Connections:
- net +3.3V: now also C1.1, C15.1, C16.1, C2.1, R1.2, R2.2, U1.8 (VDD); no longer R2.1
- net +3V3: no longer C1.1, C15.1, C16.1, C2.1, R1.2, U1.8 (VDD)
- net IMAGE_OUT_1_1-: now also J3.7 (Pin_7); no longer J3.9 (Pin_9)
- net IMAGE_OUT_2_1-: now also J3.5 (Pin_5); no longer J3.7 (Pin_7)
- net POSITION_OUT_1: now also J3.9 (Pin_9); no longer J3.5 (Pin_5)
- net VREG_AVDD_1: now also R2.1; no longer R2.2
Other:
- moved on the sheet: C11, C12, C13, C14, R2

Commit message: pin assignment done
Connections:
- net HSYNC_1: now also U3.10 (GPIO7)
- net INT_XCLK: now also U3.40 (GPIO26_ADC0)
- net PCLK_1: now also U3.41 (GPIO27_ADC1)
- net SCL_cam_1: now also U3.14 (GPIO10)
- net SDA_cam_1: now also U3.27 (GPIO16)
- net VSYNC_1: now also U3.12 (GPIO8)
- net ~{RESET_1}: now also U3.13 (GPIO9)
- no-connect marks 36 -> 34
Changed lines of the file:
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@@
 	)
 	(no_connect
-		(at 157.48 154.94)
-	)
-	(no_connect
 		(at 74.295 312.42)
 	)
@@
 	)
 	(no_connect
-		(at 157.48 157.48)
-	)
-	(no_connect
 		(at 112.395 316.23)
 	)
@@
 	(wire
 		(pts
-			(xy 153.67 86.36) (xy 168.91 86.36)
+			(xy 153.67 86.36) (xy 163.83 86.36)
 		)
 		(stroke
@@
 	)
 	(label "GPIO0_1"
-		(at 168.91 86.36 180)
+		(at 163.83 86.36 180)
 		(effects
 			(font
@@
 		)
 	)
-	(global_label "DATA5_1"
-		(shape output)
-		(at 271.78 149.86 0)
+	(global_label "~{RESET_1}"
+		(shape input)
+		(at 160.02 109.22 0)
 		(fields_autoplaced yes)
 		(effects
@@
 		)
 		(property "Intersheetrefs" "${INTERSHEET_REFS}"
-			(at 282.5666 149.86 0)
+			(at 170.9274 109.22 0)
 			(effects
 				(font
@@
 		)
 	)
-	(global_label "DATA2_1"
+	(global_label "DATA5_1"
 		(shape output)
-		(at 271.78 147.32 0)
+		(at 271.78 149.86 0)
 		(fields_autoplaced yes)
 		(effects
@@
 		)
 		(property "Intersheetrefs" "${INTERSHEET_REFS}"
-			(at 282.5666 147.32 0)
+			(at 282.5666 149.86 0)
 			(effects
 				(font
@@
 		)
 	)
-	(global_label "~{RESET_1}"
-		(shape input)
-		(at 194.31 134.62 0)
+	(global_label "DATA2_1"
+		(shape output)
+		(at 271.78 147.32 0)
 		(fields_autoplaced yes)
 		(effects
@@
 		)
 		(property "Intersheetrefs" "${INTERSHEET_REFS}"
-			(at 205.2174 134.62 0)
+			(at 282.5666 147.32 0)
 			(effects
 				(font
@@
 		)
 	)
-	(global_label "SWD_1"
+	(global_label "SCL_cam_1"
 		(shape input)
-		(at 158.75 321.31 180)
+		(at 160.02 111.76 0)
 		(fields_autoplaced yes)
 		(effects
@@
 				(size 1.27 1.27)
 			)
-			(justify right)
+			(justify left)
 		)
 		(property "Intersheetrefs" "${INTERSHEET_REFS}"
-			(at 149.6568 321.31 0)
+			(at 173.5884 111.76 0)
 			(effects
 				(font
 					(size 1.27 1.27)
 				)
-				(justify right)
+				(justify left)
 				(hide yes)
 			)
 		)
 	)
-	(global_label "SDA_cam_1"
+	(global_label "SWD_1"
 		(shape input)
-		(at 194.31 129.54 0)
+		(at 158.75 321.31 180)
 		(fields_autoplaced yes)
 		(effects
@@
 				(size 1.27 1.27)
 			)
-			(justify left)
+			(justify right)
 		)
 		(property "Intersheetrefs" "${INTERSHEET_REFS}"
-			(at 207.9389 129.54 0)
+			(at 149.6568 321.31 0)
 			(effects
 				(font
 					(size 1.27 1.27)
 				)
-				(justify left)
+				(justify right)
 				(hide yes)
 			)
@@
 	(global_label "INT_XCLK"
 		(shape input)
-		(at 176.53 147.32 0)
+		(at 157.48 154.94 0)
 		(fields_autoplaced yes)
 		(effects
@@
 		)
 		(property "Intersheetrefs" "${INTERSHEET_REFS}"
-			(at 188.1633 147.32 0)
+			(at 169.1133 154.94 0)
 			(effects
 				(font
@@
 		)
 	)
-	(global_label "VSYNC_1"
-		(shape input)
-		(at 166.37 104.14 0)
-		(fields_autoplaced yes)
-		(effects
-			(font
-				(size 1.27 1.27)
-			)
-			(justify left)
-		)
-		(property "Intersheetrefs" "${INTERSHEET_REFS}"
-			(at 177.5195 104.14 0)
-			(effects
-				(font
-					(size 1.27 1.27)
-				)
-				(justify left)
-				(hide yes)
-			)
-		)
-	)
 	(global_label "DATA7_1"
 		(shape output)
@@
 	(global_label "PCLK_1"
 		(shape input)
-		(at 194.31 127 0)
+		(at 157.48 157.48 0)
 		(fields_autoplaced yes)
 		(effects
@@
 		)
 		(property "Intersheetrefs" "${INTERSHEET_REFS}"
-			(at 204.3104 127 0)
+			(at 167.4804 157.48 0)
 			(effects
 				(font
@@
 		)
 	)
-	(global_label "SCL_cam_1"
-		(shape input)
-		(at 194.31 132.08 0)
+	(global_label "DGND"
+		(shape bidirectional)
+		(at 350.52 102.87 90)
 		(fields_autoplaced yes)
 		(effects
@@
 		)
 		(property "Intersheetrefs" "${INTERSHEET_REFS}"
-			(at 207.8784 132.08 0)
+			(at 350.52 93.633 90)
 			(effects
 				(font
@@
 		)
 	)
-	(global_label "DGND"
-		(shape bidirectional)
-		(at 350.52 102.87 90)
+	(global_label "IMAGE_OUT_1_1"
+		(shape input)
+		(at 128.905 316.23 0)
 		(fields_autoplaced yes)
 		(effects
@@
 		)
 		(property "Intersheetrefs" "${INTERSHEET_REFS}"
-			(at 350.52 93.633 90)
+			(at 146.4044 316.23 0)
 			(effects
 				(font
@@
 		)
 	)
-	(global_label "IMAGE_OUT_1_1"
-		(shape input)
-		(at 128.905 316.23 0)
+	(global_label "DATA0_1"
+		(shape output)
+		(at 271.78 160.02 0)
 		(fields_autoplaced yes)
 		(effects
@@
 		)
 		(property "Intersheetrefs" "${INTERSHEET_REFS}"
-			(at 146.4044 316.23 0)
+			(at 282.5666 160.02 0)
 			(effects
 				(font
@@
 		)
 	)
-	(global_label "DATA0_1"
-		(shape output)
-		(at 271.78 160.02 0)
+	(global_label "HSYNC_1"
+		(shape input)
+		(at 160.02 104.14 0)
 		(fields_autoplaced yes)
 		(effects
@@
 		)
 		(property "Intersheetrefs" "${INTERSHEET_REFS}"
-			(at 282.5666 160.02 0)
+			(at 171.4114 104.14 0)
 			(effects
 				(font
@@
 		)
 	)
-	(global_label "HSYNC_1"
+	(global_label "SDA_cam_1"
+		(shape input)
+		(at 160.02 127 0)
+		(fields_autoplaced yes)
+		(effects
+			(font
+				(size 1.27 1.27)
+			)
+			(justify left)
+		)
+		(property "Intersheetrefs" "${INTERSHEET_REFS}"
+			(at 173.6489 127 0)
+			(effects
+				(font
+					(size 1.27 1.27)
+				)
+				(justify left)
+				(hide yes)
+			)
+		)
+	)
+	(global_label "VSYNC_1"
 		(shape input)
-		(at 166.37 106.68 0)
+		(at 160.02 106.68 0)
 		(fields_autoplaced yes)
 		(effects
@@
 		)
 		(property "Intersheetrefs" "${INTERSHEET_REFS}"
-			(at 177.7614 106.68 0)
+			(at 171.1695 106.68 0)
 			(effects
 				(font

Commit message: finished connecting all data pins
Connections:
- net HSYNC_1: now also U3.27 (GPIO16); no longer U3.10 (GPIO7)
- net SCL_cam_1: now also U3.13 (GPIO9); no longer U3.14 (GPIO10)
- net SDA_cam_1: now also U3.14 (GPIO10); no longer U3.27 (GPIO16)
- net VSYNC_1: now also U3.10 (GPIO7); no longer U3.12 (GPIO8)
- net ~{RESET_1}: now also U3.12 (GPIO8); no longer U3.13 (GPIO9)
Changed lines of the file:
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@@
 	(global_label "~{RESET_1}"
 		(shape input)
-		(at 160.02 109.22 0)
-		(fields_autoplaced yes)
-		(effects
-			(font
-				(size 1.27 1.27)
-			)
-			(justify left)
-		)
-		(property "Intersheetrefs" "${INTERSHEET_REFS}"
-			(at 170.9274 109.22 0)
+		(at 160.02 106.68 0)
+		(fields_autoplaced yes)
+		(effects
+			(font
+				(size 1.27 1.27)
+			)
+			(justify left)
+		)
+		(property "Intersheetrefs" "${INTERSHEET_REFS}"
+			(at 170.9274 106.68 0)
 			(effects
 				(font
@@
 	(global_label "SCL_cam_1"
 		(shape input)
-		(at 160.02 111.76 0)
-		(fields_autoplaced yes)
-		(effects
-			(font
-				(size 1.27 1.27)
-			)
-			(justify left)
-		)
-		(property "Intersheetrefs" "${INTERSHEET_REFS}"
-			(at 173.5884 111.76 0)
+		(at 160.02 109.22 0)
+		(fields_autoplaced yes)
+		(effects
+			(font
+				(size 1.27 1.27)
+			)
+			(justify left)
+		)
+		(property "Intersheetrefs" "${INTERSHEET_REFS}"
+			(at 173.5884 109.22 0)
 			(effects
 				(font
@@
 	(global_label "HSYNC_1"
 		(shape input)
+		(at 160.02 127 0)
+		(fields_autoplaced yes)
+		(effects
+			(font
+				(size 1.27 1.27)
+			)
+			(justify left)
+		)
+		(property "Intersheetrefs" "${INTERSHEET_REFS}"
+			(at 171.4114 127 0)
+			(effects
+				(font
+					(size 1.27 1.27)
+				)
+				(justify left)
+				(hide yes)
+			)
+		)
+	)
+	(global_label "DATA1_1"
+		(shape output)
+		(at 271.78 157.48 0)
+		(fields_autoplaced yes)
+		(effects
+			(font
+				(size 1.27 1.27)
+			)
+			(justify left)
+		)
+		(property "Intersheetrefs" "${INTERSHEET_REFS}"
+			(at 282.5666 157.48 0)
+			(effects
+				(font
+					(size 1.27 1.27)
+				)
+				(justify left)
+				(hide yes)
+			)
+		)
+	)
+	(global_label "IMAGE_OUT_1_1+"
+		(shape output)
+		(at 160.02 124.46 0)
+		(fields_autoplaced yes)
+		(effects
+			(font
+				(size 1.27 1.27)
+			)
+			(justify left)
+		)
+		(property "Intersheetrefs" "${INTERSHEET_REFS}"
+			(at 179.0918 124.46 0)
+			(effects
+				(font
+					(size 1.27 1.27)
+				)
+				(justify left)
+				(hide yes)
+			)
+		)
+	)
+	(global_label "EXT_XCLK_1"
+		(shape input)
+		(at 298.45 129.54 0)
+		(fields_autoplaced yes)
+		(effects
+			(font
+				(size 1.27 1.27)
+			)
+			(justify left)
+		)
+		(property "Intersheetrefs" "${INTERSHEET_REFS}"
+			(at 312.6836 129.54 0)
+			(effects
+				(font
+					(size 1.27 1.27)
+				)
+				(justify left)
+				(hide yes)
+			)
+		)
+	)
+	(global_label "DATA3_1"
+		(shape output)
+		(at 271.78 152.4 0)
+		(fields_autoplaced yes)
+		(effects
+			(font
+				(size 1.27 1.27)
+			)
+			(justify left)
+		)
+		(property "Intersheetrefs" "${INTERSHEET_REFS}"
+			(at 282.5666 152.4 0)
+			(effects
+				(font
+					(size 1.27 1.27)
+				)
+				(justify left)
+				(hide yes)
+			)
+		)
+	)
+	(global_label "SDA_cam_1"
+		(shape input)
+		(at 160.02 111.76 0)
+		(fields_autoplaced yes)
+		(effects
+			(font
+				(size 1.27 1.27)
+			)
+			(justify left)
+		)
+		(property "Intersheetrefs" "${INTERSHEET_REFS}"
+			(at 173.6489 111.76 0)
+			(effects
+				(font
+					(size 1.27 1.27)
+				)
+				(justify left)
+				(hide yes)
+			)
+		)
+	)
+	(global_label "VSYNC_1"
+		(shape input)
 		(at 160.02 104.14 0)
 		(fields_autoplaced yes)
@@
 		)
 		(property "Intersheetrefs" "${INTERSHEET_REFS}"
-			(at 171.4114 104.14 0)
-			(effects
-				(font
-					(size 1.27 1.27)
-				)
-				(justify left)
-				(hide yes)
-			)
-		)
-	)
-	(global_label "DATA1_1"
-		(shape output)
-		(at 271.78 157.48 0)
-		(fields_autoplaced yes)
-		(effects
-			(font
-				(size 1.27 1.27)
-			)
-			(justify left)
-		)
-		(property "Intersheetrefs" "${INTERSHEET_REFS}"
-			(at 282.5666 157.48 0)
-			(effects
-				(font
-					(size 1.27 1.27)
-				)
-				(justify left)
-				(hide yes)
-			)
-		)
-	)
-	(global_label "IMAGE_OUT_1_1+"
-		(shape output)
-		(at 160.02 124.46 0)
-		(fields_autoplaced yes)
-		(effects
-			(font
-				(size 1.27 1.27)
-			)
-			(justify left)
-		)
-		(property "Intersheetrefs" "${INTERSHEET_REFS}"
-			(at 179.0918 124.46 0)
-			(effects
-				(font
-					(size 1.27 1.27)
-				)
-				(justify left)
-				(hide yes)
-			)
-		)
-	)
-	(global_label "EXT_XCLK_1"
-		(shape input)
-		(at 298.45 129.54 0)
-		(fields_autoplaced yes)
-		(effects
-			(font
-				(size 1.27 1.27)
-			)
-			(justify left)
-		)
-		(property "Intersheetrefs" "${INTERSHEET_REFS}"
-			(at 312.6836 129.54 0)
-			(effects
-				(font
-					(size 1.27 1.27)
-				)
-				(justify left)
-				(hide yes)
-			)
-		)
-	)
-	(global_label "DATA3_1"
-		(shape output)
-		(at 271.78 152.4 0)
-		(fields_autoplaced yes)
-		(effects
-			(font
-				(size 1.27 1.27)
-			)
-			(justify left)
-		)
-		(property "Intersheetrefs" "${INTERSHEET_REFS}"
-			(at 282.5666 152.4 0)
-			(effects
-				(font
-					(size 1.27 1.27)
-				)
-				(justify left)
-				(hide yes)
-			)
-		)
-	)
-	(global_label "SDA_cam_1"
-		(shape input)
-		(at 160.02 127 0)
-		(fields_autoplaced yes)
-		(effects
-			(font
-				(size 1.27 1.27)
-			)
-			(justify left)
-		)
-		(property "Intersheetrefs" "${INTERSHEET_REFS}"
-			(at 173.6489 127 0)
-			(effects
-				(font
-					(size 1.27 1.27)
-				)
-				(justify left)
-				(hide yes)
-			)
-		)
-	)
-	(global_label "VSYNC_1"
-		(shape input)
-		(at 160.02 106.68 0)
-		(fields_autoplaced yes)
-		(effects
-			(font
-				(size 1.27 1.27)
-			)
-			(justify left)
-		)
-		(property "Intersheetrefs" "${INTERSHEET_REFS}"
-			(at 171.1695 106.68 0)
-			(effects
-				(font
+			(at 171.1695 104.14 0)
+			(effects
+				(font

Commit message: layout finalized (?)
Parts:
- R1: footprint Capacitor_SMD:C_0402_1005Metric -> Resistor_SMD:R_0402_1005Metric_Pad0.72x0.64mm_HandSolder
- R10, R11, R12, R13, R14, R15, R16, R17, R2, R3, R4, R6, R9: footprint Capacitor_SMD:C_0402_1005Metric -> Resistor_SMD:R_0402_1005Metric
- R18, R19, R20, R21: footprint Resistor_SMD:R_0603_1608Metric_Pad0.98x0.95mm_HandSolder -> Resistor_SMD:R_0402_1005Metric
Connections:
- net +3V3 is gone; now on net +3.3V: U1.5 (VDDIO)
- net GND: now also J2.8 (Pin_8); no longer J2.5 (Pin_5)
- net SWCLK_1: now also J2.5 (Pin_5)
- net SWD_1: now also J2.7 (Pin_7)
- no-connect marks 34 -> 37
Other:
- moved on the sheet: C1, C15, C16, C2, R1, U1

Commit message: minor changes
Parts:
- added C32: 100n, Capacitor_SMD:C_0402_1005Metric, symbol Device:C
Connections:
- net +3.3V: now also C32.1
- net GND: now also C32.2
Changed lines of the file:
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@@
 	(wire
 		(pts
+			(xy 316.23 125.73) (xy 316.23 129.54)
+		)
+		(stroke
+			(width 0)
+			(type default)
+		)
+	)
+	(wire
+		(pts
 			(xy 105.41 261.62) (xy 104.14 261.62)
 		)
@@
 	(wire
 		(pts
+			(xy 316.23 115.57) (xy 316.23 118.11)
+		)
+		(stroke
+			(width 0)
+			(type default)
+		)
+	)
+	(wire
+		(pts
 			(xy 153.67 149.86) (xy 160.02 149.86)
 		)
@@
 	)
 	(symbol
+		(lib_name "GND_8")
+		(lib_id "power:GND")
+		(at 316.23 129.54 0)
+		(unit 1)
+		(exclude_from_sim no)
+		(in_bom yes)
+		(on_board yes)
+		(dnp no)
+		(fields_autoplaced yes)
+		(property "Reference" "#PWR064"
+			(at 316.23 135.89 0)
+			(effects
+				(font
+					(size 1.27 1.27)
+				)
+				(hide yes)
+			)
+		)
+		(property "Value" "GND"
+			(at 316.23 134.62 0)
+			(effects
+				(font
+					(size 1.27 1.27)
+				)
+				(hide yes)
+			)
+		)
+		(property "Footprint" ""
+			(at 316.23 129.54 0)
+			(effects
+				(font
+					(size 1.27 1.27)
+				)
+				(hide yes)
+			)
+		)
+		(property "Datasheet" ""
+			(at 316.23 129.54 0)
+			(effects
+				(font
+					(size 1.27 1.27)
+				)
+				(hide yes)
+			)
+		)
+		(property "Description" "Power symbol creates a global label with name \"GND\" , ground"
+			(at 316.23 129.54 0)
+			(effects
+				(font
+					(size 1.27 1.27)
+				)
+				(hide yes)
+			)
+		)
+		(pin "1"
+		)
+		(instances
+			(project "FPSP Camera"
+				(path "/b8279e3f-7ea4-46f5-abf2-a9173e16562f"
+					(reference "#PWR064")
+					(unit 1)
+				)
+			)
+		)
+	)
+	(symbol
 		(lib_id "Device:R")
 		(at 72.39 69.85 270)
@@
 	)
 	(symbol
+		(lib_id "power:+3.3V")
+		(at 316.23 115.57 0)
+		(unit 1)
+		(exclude_from_sim no)
+		(in_bom yes)
+		(on_board yes)
+		(dnp no)
+		(fields_autoplaced yes)
+		(property "Reference" "#PWR063"
+			(at 316.23 119.38 0)
+			(effects
+				(font
+					(size 1.27 1.27)
+				)
+				(hide yes)
+			)
+		)
+		(property "Value" "+3.3V"
+			(at 316.23 110.49 0)
+			(effects
+				(font
+					(size 1.27 1.27)
+				)
+			)
+		)
+		(property "Footprint" ""
+			(at 316.23 115.57 0)
+			(effects
+				(font
+					(size 1.27 1.27)
+				)
+				(hide yes)
+			)
+		)
+		(property "Datasheet" ""
+			(at 316.23 115.57 0)
+			(effects
+				(font
+					(size 1.27 1.27)
+				)
+				(hide yes)
+			)
+		)
+		(property "Description" "Power symbol creates a global label with name \"+3.3V\""
+			(at 316.23 115.57 0)
+			(effects
+				(font
+					(size 1.27 1.27)
+				)
+				(hide yes)
+			)
+		)
+		(pin "1"
+		)
+		(instances
+			(project "FPSP Camera"
+				(path "/b8279e3f-7ea4-46f5-abf2-a9173e16562f"
+					(reference "#PWR063")
+					(unit 1)
+				)
+			)
+		)
+	)
+	(symbol
 		(lib_id "Device:R")
 		(at 337.82 139.7 270)
@@
 					(unit 1)
 				)
+			)
+		)
+	)
+	(symbol
+		(lib_id "Device:C")
+		(at 316.23 121.92 0)
+		(unit 1)
+		(exclude_from_sim no)
+		(in_bom yes)
+		(on_board yes)
+		(dnp no)
+		(property "Reference" "C32"
+			(at 319.151 120.7516 0)
+			(effects
+				(font
+					(size 1.27 1.27)
+				)
+				(justify left)
+			)
+		)
+		(property "Value" "100n"
+			(at 319.151 123.063 0)
+			(effects
+				(font
+					(size 1.27 1.27)
+				)
+				(justify left)
+			)
+		)
+		(property "Footprint" "Capacitor_SMD:C_0402_1005Metric"
+			(at 317.1952 125.73 0)
+			(effects
+				(font
+					(size 1.27 1.27)
+				)
+				(hide yes)
+			)
+		)
+		(property "Datasheet" "~"
+			(at 316.23 121.92 0)
+			(effects
+				(font
+					(size 1.27 1.27)
+				)
+				(hide yes)
+			)
+		)
+		(property "Description" ""
+			(at 316.23 121.92 0)
+			(effects
+				(font
+					(size 1.27 1.27)
+				)
+			)
+		)
+		(pin "1"
+		)
+		(pin "2"
+		)
+		(instances
+			(project "FPSP Camera"
+				(path "/b8279e3f-7ea4-46f5-abf2-a9173e16562f"
+					(reference "C32")
+					(unit 1)
+				)

Commit message: '
Parts:
- added J7: Conn_01x02, Connector_PinHeader_2.54mm:PinHeader_1x02_P2.54mm_Vertical, symbol Connector_Generic:Conn_01x02
Connections:
- net +5V: now also J7.1 (Pin_1)
- net GND: now also J7.2 (Pin_2)
Other:
- note added: "Power"
Changed lines of the file:
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@@
 	)
 	(rectangle
+		(start 158.75 242.57)
+		(end 203.2 275.59)
+		(stroke
+			(width 0)
+			(type default)
+		)
+		(fill
+			(type none)
+		)
+	)
+	(rectangle
 		(start 254 88.9)
 		(end 359.41 180.34)
@@
 		)
 	)
+	(text "Power"
+		(exclude_from_sim no)
+		(at 192.278 272.034 0)
+		(effects
+			(font
+				(size 3.81 3.81)
+				(thickness 0.4763)
+				(italic yes)
+			)
+		)
+	)
 	(text "2.8 V"
 		(exclude_from_sim no)
@@
 	(wire
 		(pts
+			(xy 165.1 256.54) (xy 167.64 256.54)
+		)
+		(stroke
+			(width 0)
+			(type default)
+		)
+	)
+	(wire
+		(pts
 			(xy 87.63 80.01) (xy 90.17 80.01)
 		)
@@
 	(wire
 		(pts
+			(xy 165.1 254) (xy 167.64 254)
+		)
+		(stroke
+			(width 0)
+			(type default)
+		)
+	)
+	(wire
+		(pts
 			(xy 52.07 97.79) (xy 67.945 97.79)
 		)
@@
 	)
 	(symbol
+		(lib_id "power:GND")
+		(at 165.1 256.54 0)
+		(unit 1)
+		(exclude_from_sim no)
+		(in_bom yes)
+		(on_board yes)
+		(dnp no)
+		(fields_autoplaced yes)
+		(property "Reference" "#PWR066"
+			(at 165.1 262.89 0)
+			(effects
+				(font
+					(size 1.27 1.27)
+				)
+				(hide yes)
+			)
+		)
+		(property "Value" "GND"
+			(at 165.1 261.62 0)
+			(effects
+				(font
+					(size 1.27 1.27)
+				)
+				(hide yes)
+			)
+		)
+		(property "Footprint" ""
+			(at 165.1 256.54 0)
+			(effects
+				(font
+					(size 1.27 1.27)
+				)
+				(hide yes)
+			)
+		)
+		(property "Datasheet" ""
+			(at 165.1 256.54 0)
+			(effects
+				(font
+					(size 1.27 1.27)
+				)
+				(hide yes)
+			)
+		)
+		(property "Description" "Power symbol creates a global label with name \"GND\" , ground"
+			(at 165.1 256.54 0)
+			(effects
+				(font
+					(size 1.27 1.27)
+				)
+				(hide yes)
+			)
+		)
+		(pin "1"
+		)
+		(instances
+			(project "FPSP Camera"
+				(path "/b8279e3f-7ea4-46f5-abf2-a9173e16562f"
+					(reference "#PWR066")
+					(unit 1)
+				)
+			)
+		)
+	)
+	(symbol
 		(lib_id "Device:C")
 		(at 90.17 40.64 0)
@@
 	)
 	(symbol
+		(lib_id "power:+5V")
+		(at 165.1 254 0)
+		(unit 1)
+		(exclude_from_sim no)
+		(in_bom yes)
+		(on_board yes)
+		(dnp no)
+		(fields_autoplaced yes)
+		(property "Reference" "#PWR065"
+			(at 165.1 257.81 0)
+			(effects
+				(font
+					(size 1.27 1.27)
+				)
+				(hide yes)
+			)
+		)
+		(property "Value" "+5V"
+			(at 165.1 248.92 0)
+			(effects
+				(font
+					(size 1.27 1.27)
+				)
+			)
+		)
+		(property "Footprint" ""
+			(at 165.1 254 0)
+			(effects
+				(font
+					(size 1.27 1.27)
+				)
+				(hide yes)
+			)
+		)
+		(property "Datasheet" ""
+			(at 165.1 254 0)
+			(effects
+				(font
+					(size 1.27 1.27)
+				)
+				(hide yes)
+			)
+		)
+		(property "Description" "Power symbol creates a global label with name \"+5V\""
+			(at 165.1 254 0)
+			(effects
+				(font
+					(size 1.27 1.27)
+				)
+				(hide yes)
+			)
+		)
+		(pin "1"
+		)
+		(instances
+			(project "FPSP Camera"
+				(path "/b8279e3f-7ea4-46f5-abf2-a9173e16562f"
+					(reference "#PWR065")
+					(unit 1)
+				)
+			)
+		)
+	)
+	(symbol
 		(lib_id "power:GND")
 		(at 382.27 50.8 0)
@@
 					(unit 1)
 				)
+			)
+		)
+	)
+	(symbol
+		(lib_id "Connector_Generic:Conn_01x02")
+		(at 172.72 254 0)
+		(unit 1)
+		(exclude_from_sim no)
+		(in_bom yes)
+		(on_board yes)
+		(dnp no)
+		(fields_autoplaced yes)
+		(property "Reference" "J7"
+			(at 175.26 253.9999 0)
+			(effects
+				(font
+					(size 1.27 1.27)
+				)
+				(justify left)
+			)
+		)
+		(property "Value" "Conn_01x02"
+			(at 175.26 256.5399 0)
+			(effects
+				(font
+					(size 1.27 1.27)
+				)
+				(justify left)
+			)
+		)
+		(property "Footprint" "Connector_PinHeader_2.54mm:PinHeader_1x02_P2.54mm_Vertical"
+			(at 172.72 254 0)
+			(effects
+				(font
+					(size 1.27 1.27)
+				)
+				(hide yes)
+			)
+		)
+		(property "Datasheet" "~"
+			(at 172.72 254 0)
+			(effects
+				(font
+					(size 1.27 1.27)
+				)
+				(hide yes)
+			)
+		)
+		(property "Description" "Generic connector, single row, 01x02, script generated (kicad-library-utils/schlib/autogen/connector/)"
+			(at 172.72 254 0)
+			(effects
+				(font
+					(size 1.27 1.27)
+				)
+				(hide yes)
+			)
+		)
+		(pin "1"
+		)
+		(pin "2"
+		)
+		(instances
+			(project ""
+				(path "/b8279e3f-7ea4-46f5-abf2-a9173e16562f"
+					(reference "J7")
+					(unit 1)
+				)

Commit message: FPC socket foorprint replaced
Parts:
- J1: footprint Connector_FFC-FPC:TE_2-1734839-3_1x23-1MP_P0.5mm_Horizontal -> 52435-2471:MOLEX_52435-2471
Changed lines of the file:
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@@
 			)
 		)
-		(property "Footprint" "Connector_FFC-FPC:TE_2-1734839-3_1x23-1MP_P0.5mm_Horizontal"
+		(property "Footprint" "52435-2471:MOLEX_52435-2471"
 			(at 266.7 129.54 0)
 			(effects
