File: FPSP Camera.kicad_sch (KiCad schematic)
At the start: 80 parts, among them J1 Conn_01x24_Socket, J2 Conn_02x04_Counter_Clockwise, J3 Conn_02x07_Counter_Clockwise, J4 SM03B-SRSS-TB, J5 USB_B_Micro, J6 Conn_02x06_Odd_Even, J7 Conn_01x02, U1 ICM-45686, U2 W25Q128JVS, U3 RP2350_60QFN, U4 TLV75533PDRV, U5 TLV73328PDRV, U6 TLV73315PDRV, Y1 SiT8008xx-1x-xxE

Commit message: test PCB version 2 completed
Parts:
- removed J2: Conn_02x04_Counter_Clockwise, Connector_Molex:Molex_SlimStack_502426-0810_2x04_P0.40mm_Vertical, symbol Connector_Generic:Conn_02x04_Odd_Even
- added J3: Conn_02x07_Counter_Clockwise, Connector_Molex:Molex_SlimStack_502426-1410_2x07_P0.40mm_Vertical, symbol Connector_Generic:Conn_02x07_Odd_Even
- added TP2: TestPoint, TestPoint:TestPoint_Pad_D1.0mm, symbol Connector:TestPoint
- renumbered C3 to C1, C4 to C2, C32 to C23, C23 to C24, C24 to C25, C25 to C26, C26 to C27, C27 to C28, C28 to C29, C5 to C3, C29 to C30, C30 to C31, C31 to C32, C1 to C4, C2 to C5, J7 to J2, J3 to J4, J4 to J5, J5 to J6, J6 to J7
Connections:
- net +5V: now also J3.2 (Pin_2)
- net DATA3_1: now also U3.35 (GPIO23); no longer U3.36 (GPIO24)
- net DATA4_1: now also U3.36 (GPIO24); no longer U3.37 (GPIO25)
- net DATA5_1: now also U3.37 (GPIO25); no longer U3.35 (GPIO23)
- net DATA6_1: now also U3.40 (GPIO26_ADC0); no longer U3.33 (GPIO21)
- net DATA7_1: now also U3.41 (GPIO27_ADC1); no longer U3.32 (GPIO20)
- net DATA8_1: now also U3.42 (GPIO28_ADC2); no longer U3.31 (GPIO19)
- net DATA9_1: now also U3.43 (GPIO29_ADC3); no longer U3.28 (GPIO17)
- net EXT_XCLK_1: now also TP2.1; no longer U3.29 (GPIO18)
- net GND: now also J4.14 (Pin_14), J3.14 (Pin_14); no longer J4.11 (Pin_11)
- net HSYNC_1: now also U3.9 (GPIO6); no longer U3.27 (GPIO16)
- net INT_XCLK: now also U3.33 (GPIO21); no longer U3.40 (GPIO26_ADC0)
- net PCLK_1: now also U3.8 (GPIO5); no longer U3.41 (GPIO27_ADC1)
- net POSITION_OUT_1: now also J4.3 (Pin_3), U3.31 (GPIO19); no longer J4.9 (Pin_9), U3.15 (GPIO11)
- net SWCLK_1: now also J3.5 (Pin_5)
- net SWD_1: now also J3.7 (Pin_7)
- net USB_D1+: now also J3.1 (Pin_1)
- net USB_D1-: now also J3.3 (Pin_3)
- net FPGA_EN: now reaches J4.13 (Pin_13)
- net FPGA_EN: now also U3.15 (GPIO11)
- net IMAGE_CLK: now reaches J4.4 (Pin_4)
- net IMAGE_CLK: now also U3.27 (GPIO16)
- net VSYNC_OUT: now reaches J4.6 (Pin_6)
- net VSYNC_OUT: now also U3.28 (GPIO17)
- net POSITION_OUT_CLK: now reaches J4.8 (Pin_8)
- net POSITION_OUT_CLK: now also U3.29 (GPIO18)
- net IMAGE_OUT_1_1+ renamed HREF_OUT
- net HREF_OUT: now also U3.32 (GPIO20); no longer U3.19 (GPIO15)
- net IMAGE_OUT_1_1- renamed IMAGE_OUT_1
- net IMAGE_OUT_1: now also J4.11 (Pin_11); no longer J4.7 (Pin_7)
- net IMAGE_OUT_2_1+ renamed IMAGE_OUT_3
- net IMAGE_OUT_3: now also J4.7 (Pin_7); no longer J4.3 (Pin_3)
- net IMAGE_OUT_2_1- renamed IMAGE_OUT_2
- net IMAGE_OUT_2: now also J4.9 (Pin_9); no longer J4.5 (Pin_5)
- new net IMAGE_OUT_4: J4.5 (Pin_5), U3.19 (GPIO15)
- no-connect marks 37 -> 33
Other:
- note removed: "HSTX: 12-19"
- moved on the sheet: J4

Commit message: refined 5V net isolation
Connections:
- net +5V: no longer J3.2 (Pin_2)
- no-connect marks 33 -> 34
Changed lines of the file:
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@@
 	)
 	(no_connect
+		(at 57.15 255.27)
+	)
+	(no_connect
 		(at 336.55 52.07)
 	)
@@
 	(wire
 		(pts
-			(xy 55.88 255.27) (xy 59.69 255.27)
-		)
-		(stroke
-			(width 0)
-			(type default)
-		)
-	)
-	(wire
-		(pts
 			(xy 196.85 156.21) (xy 196.85 157.48)
 		)
@@
 	(wire
 		(pts
+			(xy 55.88 255.27) (xy 57.15 255.27)
+		)
+		(stroke
+			(width 0)
+			(type default)
+		)
+	)
+	(wire
+		(pts
 			(xy 45.72 208.28) (xy 43.18 208.28)
 		)
@@
 					(unit 1)
 				)
-			)
-		)
-	)
-	(symbol
-		(lib_id "power:+5V")
-		(at 59.69 255.27 0)
-		(unit 1)
-		(body_style 1)
-		(exclude_from_sim no)
-		(in_bom yes)
-		(on_board yes)
-		(in_pos_files yes)
-		(dnp no)
-		(fields_autoplaced yes)
-		(property "Reference" "#PWR067"
-			(at 59.69 259.08 0)
-			(hide yes)
-			(show_name no)
-			(do_not_autoplace no)
-			(effects
-				(font
-					(size 1.27 1.27)
-				)
-			)
-		)
-		(property "Value" "+5V"
-			(at 59.69 250.19 0)
-			(show_name no)
-			(do_not_autoplace no)
-			(effects
-				(font
-					(size 1.27 1.27)
-				)
-			)
-		)
-		(property "Footprint" ""
-			(at 59.69 255.27 0)
-			(hide yes)
-			(show_name no)
-			(do_not_autoplace no)
-			(effects
-				(font
-					(size 1.27 1.27)
-				)
-			)
-		)
-		(property "Datasheet" ""
-			(at 59.69 255.27 0)
-			(hide yes)
-			(show_name no)
-			(do_not_autoplace no)
-			(effects
-				(font
-					(size 1.27 1.27)
-				)
-			)
-		)
-		(property "Description" "Power symbol creates a global label with name \"+5V\""
-			(at 59.69 255.27 0)
-			(hide yes)
-			(show_name no)
-			(do_not_autoplace no)
-			(effects
-				(font
-					(size 1.27 1.27)
-				)
-			)
-		)
-		(pin "1"
-		)
-		(instances
-			(project "FPSP Camera"
-				(path "/b8279e3f-7ea4-46f5-abf2-a9173e16562f"
-					(reference "#PWR067")
-					(unit 1)
-				)
