File: FPSP Camera.kicad_pcb (KiCad board)
At the start: 4 copper layers, 85.7 x 35 mm, 70 parts, among them J4 Conn_01x24_Socket, U1 TLV75533PDRV, U2 TLV73328PDRV, U3 RP2350_60QFN, U4 TLV73315PDRV, U6 ICM-45686, Y1 SiT8008xx-1x-xxE

Commit message: connector PCB added
Parts:
- added J5: Conn_02x04_Counter_Clockwise, Connector_Molex:Molex_SlimStack_502426-0810_2x04_P0.40mm_Vertical, F.Cu at (46.7, 52.8)
- added J6: Conn_02x07_Counter_Clockwise, Connector_Molex:Molex_SlimStack_502426-1410_2x07_P0.40mm_Vertical, F.Cu at (59.4, 45.0)
- R10, R11, R12, R15: footprint Capacitor_SMD:C_0402_1005Metric -> Resistor_SMD:R_0603_1608Metric_Pad0.98x0.95mm_HandSolder
Connections:
- U3 pad 15: unconnected-(U3-GPIO11-Pad15) -> POSITION_OUT_1
- U3 pad 16: IMAGE_OUT_1_1+ -> IMAGE_OUT_1_1-
- U3 pad 17: IMAGE_OUT_1_1- -> IMAGE_OUT_2_1-
- U3 pad 19: IMAGE_OUT_2_1- -> IMAGE_OUT_1_1+
- U3 pad 27: POSITION_OUT_1 -> unconnected-(U3-GPIO16-Pad27)
Routing:
- net IMAGE_OUT_2_1-: track 2.08 -> 3.11 mm
- net IMAGE_OUT_1_1+: track 2.70 -> 2.08 mm

Commit message: routing updates
Parts:
- removed the C19 at (64.9, 22.2)
- removed R115: 0R, Resistor_SMD:R_0603_1608Metric_Pad0.98x0.95mm_HandSolder
- L1: footprint Inductor_SMD:L_1210_3225Metric -> Inductor_SMD:L_pol_2016
- moved JP3 105.3 mm to (79.8, 24.8)
- moved C21 88.9 mm to (85.8, 29.8)
- moved C22 88.5 mm to (85.8, 30.8)
- moved J2 43.5 mm to (67.4, 14.6), turned to 180 degrees
- moved R2 22.5 mm to (71.5, 22.5), turned to 90 degrees
- moved TP1 22.3 mm to (71.3, 20.0)
- moved C18 22.2 mm to (69.3, 24.8)
- moved L1 20.2 mm to (69.3, 22.0), turned to 0 degrees
- moved C19 19.0 mm to (69.3, 23.8), turned to 0 degrees
- moved C17 17.8 mm to (71.5, 24.5), turned to -90 degrees
- moved C14 15.2 mm to (60.8, 34.0)
- moved C4 9.15 mm to (61.5, 26.8)
- moved J3 7.90 mm to (67.3, 45.3)
- moved JP1 6.53 mm to (64.0, 20.0), turned to 180 degrees
- moved JP2 6.15 mm to (68.8, 40.5)
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- renumbered C27 to C1, C16 to C10, C20 to C11, C21 to C12, C23 to C13, C24 to C14, C28 to C15, C30 to C16, C7 to C17, C2 to C18, C3 to C19, C29 to C2, C31 to C21, C32 to C22, C26 to C23, C25 to C24, C18 to C25, C1 to C26, C5 to C27, C9 to C28, C10 to C29, C4 to C3, C13 to C30, C17 to C31, C6 to C4, C8 to C5, C11 to C6, C12 to C7, C14 to C8, C15 to C9, J4 to J1, J5 to J2, J6 to J3, R16 to R1, R4 to R10, R13 to R11, R18 to R12, R14 to R13, R19 to R14, R3 to R15, R20 to R16, R22 to R17, R10 to R18, R11 to R19, R12 to R20, R15 to R21, R5 to R3, R6 to R4, R1 to R6, R17 to R9, U6 to U1, U1 to U4, U2 to U5, U4 to U6
Connections:
- C1 pad 1: +3V3 -> +3.3V
- C15 pad 1: +3V3 -> +3.3V
- C16 pad 1: +3V3 -> +3.3V
- C2 pad 1: +3V3 -> +3.3V
- J3 pad 5: POSITION_OUT_1 -> IMAGE_OUT_2_1-
- J3 pad 7: IMAGE_OUT_2_1- -> IMAGE_OUT_1_1-
- J3 pad 9: IMAGE_OUT_1_1- -> POSITION_OUT_1
- R1 pad 2: +3V3 -> +3.3V
- R2 pad 1: +3.3V -> /VREG_AVDD_1
- R2 pad 2: /VREG_AVDD_1 -> +3.3V
- U1 pad 8: +3V3 -> +3.3V
Routing:
- net AGND: track 0.00 -> 40.6 mm, vias 0 -> 15
- net +3.3V: track 22.7 -> 61.2 mm, vias 0 -> 2
- net +1V1: track 20.2 -> 38.6 mm, vias 8 -> 9
- net /XIN_mem1: track 0.00 -> 13.2 mm, vias 0 -> 2
- net POSITION_OUT_1: track 0.00 -> 12.6 mm
- net IMAGE_OUT_1_1+: track 2.08 -> 12.2 mm
- net IMAGE_OUT_2_1+: track 2.29 -> 12.2 mm
- net IMAGE_OUT_1_1-: track 2.70 -> 12.1 mm
- net IMAGE_OUT_2_1-: track 3.11 -> 12.2 mm
- net /VREG_LX_1: track 0.00 -> 6.24 mm
- net /USB_D1-: track 0.00 -> 6.09 mm
- net /USB_D1+: track 0.00 -> 6.09 mm
- net +3V3: track 8.29 -> 3.02 mm
- net /VREG_AVDD_1: track 0.00 -> 5.14 mm
- net Net-(U3-USB_DP): track 0.00 -> 4.50 mm
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Other:
- board text added: "camera"

Commit message: pin assignment done
Parts:
- moved J1 12.9 mm to (88.5, 28.7)
- moved C31 5.59 mm to (34.4, 36.0)
- moved C26 5.59 mm to (39.2, 27.0)
- moved C27 5.59 mm to (34.2, 27.0)
- moved C28 5.59 mm to (39.2, 31.4)
- moved C30 5.59 mm to (39.1, 36.0)
- moved D1 5.59 mm to (26.7, 27.0)
- moved D2 5.59 mm to (26.6, 30.0)
- moved R18 5.59 mm to (29.9, 27.0)
- moved R19 5.59 mm to (29.9, 30.0)
- moved U4 5.59 mm to (36.7, 27.1)
- moved U6 5.59 mm to (36.6, 35.8)
- moved C29 5.59 mm to (34.5, 31.4)
- moved D3 5.59 mm to (26.7, 33.0)
- moved D4 5.59 mm to (26.7, 36.0)
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Connections:
- U3 pad 10: unconnected-(U3-GPIO7-Pad10) -> HSYNC_1
- U3 pad 12: unconnected-(U3-GPIO8-Pad12) -> VSYNC_1
- U3 pad 13: unconnected-(U3-GPIO9-Pad13) -> ~{RESET_1}
- U3 pad 14: unconnected-(U3-GPIO10-Pad14) -> SCL_cam_1
- U3 pad 27: unconnected-(U3-GPIO16-Pad27) -> SDA_cam_1
- U3 pad 40: unconnected-(U3-GPIO26_ADC0-Pad40) -> INT_XCLK
- U3 pad 41: unconnected-(U3-GPIO27_ADC1-Pad41) -> PCLK_1
Routing:
- net /USB_D1-: track 6.09 -> 1.94 mm
- net /USB_D1+: track 6.09 -> 1.94 mm
- net AGND: track 40.6 -> 37.4 mm, vias 15 -> 14
- net /~{USB_BOOT_1}: track 1.83 -> 3.45 mm
- net IMAGE_OUT_1_1-: track 12.1 -> 10.9 mm
- net POSITION_OUT_1: track 12.6 -> 11.4 mm
- net IMAGE_OUT_1_1+: track 12.2 -> 11.0 mm
- net IMAGE_OUT_2_1-: track 12.2 -> 10.9 mm
- net IMAGE_OUT_2_1+: track 12.2 -> 11.0 mm
- net HSYNC_1: track 0.00 -> 1.21 mm, vias 0 -> 1
- net +1V1: track 38.6 -> 39.4 mm
Other:
- board size 85.7 x 35 mm -> 85.7 x 30 mm

Commit message: finished connecting all data pins
Parts:
- moved J1 12.7 mm to (75.8, 30.3)
- moved C22 8.29 mm to (78.5, 34.8), turned to -90 degrees
- moved C21 7.57 mm to (78.5, 32.0), turned to -90 degrees
Connections:
- U3 pad 10: HSYNC_1 -> VSYNC_1
- U3 pad 12: VSYNC_1 -> ~{RESET_1}
- U3 pad 13: ~{RESET_1} -> SCL_cam_1
- U3 pad 14: SCL_cam_1 -> SDA_cam_1
- U3 pad 27: SDA_cam_1 -> HSYNC_1
Routing:
- net EXT_XCLK_1: track 1.72 -> 28.9 mm, vias 1 -> 2
- net SDA_cam_1: track 2.91 -> 29.0 mm, vias 1 -> 2
- net ~{RESET_1}: track 4.04 -> 28.0 mm, vias 1 -> 2
- net SCL_cam_1: track 2.91 -> 26.0 mm, vias 1 -> 2
- net INT_XCLK: track 0.00 -> 23.1 mm, vias 0 -> 2
- net VSYNC_1: track 0.00 -> 20.2 mm, vias 0 -> 1
- net PCLK_1: track 2.91 -> 16.7 mm, vias 1 -> 3
- net HSYNC_1: track 1.21 -> 13.4 mm
- net +2V8: track 4.68 -> 7.60 mm, vias 0 -> 1
- net +1V5: track 3.90 -> 5.33 mm, vias 0 -> 1
- net DATA8_1: track 11.4 -> 10.5 mm

Commit message: layout finalized (?)
Parts:
- R1: footprint Capacitor_SMD:C_0402_1005Metric -> Resistor_SMD:R_0402_1005Metric_Pad0.72x0.64mm_HandSolder
- R10, R11, R12, R13, R14, R15, R16, R17, R2, R3, R4, R6, R9: footprint Capacitor_SMD:C_0402_1005Metric -> Resistor_SMD:R_0402_1005Metric
- R18, R19, R20, R21: footprint Resistor_SMD:R_0603_1608Metric_Pad0.98x0.95mm_HandSolder -> Resistor_SMD:R_0402_1005Metric
- moved JP2 4.84 mm to (73.3, 42.2)
- moved R15 3.67 mm to (70.4, 41.3), turned to 0 degrees
- moved C22 0.85 mm to (77.8, 34.4), turned to 0 degrees
- moved C14 0.47 mm to (60.3, 34.2)
Connections:
- J2 pad 5: AGND -> SWCLK_1
- J2 pad 7: unconnected-(J2-Pin_7-Pad7) -> SWD_1
- J2 pad 8: unconnected-(J2-Pin_8-Pad8) -> AGND
- U1 pad 5: +3V3 -> +3.3V
Routing:
- net +3.3V: track 61.5 -> 148.0 mm, vias 2 -> 4
- net SWD_1: track 0.00 -> 68.4 mm, vias 0 -> 1
- net SWCLK_1: track 0.00 -> 68.1 mm, vias 0 -> 2
- net +1V5: track 5.33 -> 72.3 mm, vias 1 -> 2
- net +2V8: track 7.60 -> 63.3 mm, vias 1 -> 3
- net DGND: track 0.00 -> 16.1 mm, vias 0 -> 1
- net /RUN_1: track 4.62 -> 8.87 mm
- net +3V3: track 3.02 -> 0.00 mm
- net +1V1: track 39.5 -> 40.1 mm
- net EXT_XCLK_1: track 28.9 -> 28.3 mm
- added copper zone on B.Cu, net AGND

Commit message: minor changes
Parts:
- added C32: 100n, Capacitor_SMD:C_0402_1005Metric, F.Cu at (78.5, 30.0)
- moved C22 0.44 mm to (78.0, 34.8), turned to -90 degrees
Routing:
- net +3.3V: track 148.0 -> 160.4 mm
- net +2V8: track 63.3 -> 64.1 mm
