File: FPSP Camera.kicad_pcb (KiCad board)
At the start: 4 copper layers, 85.7 x 30 mm, 71 parts, among them J1 Conn_01x24_Socket, J2 Conn_02x04_Counter_Clockwise, J3 Conn_02x07_Counter_Clockwise, U1 ICM-45686, U3 RP2350_60QFN, U4 TLV75533PDRV, U5 TLV73328PDRV, U6 TLV73315PDRV, Y1 SiT8008xx-1x-xxE

Commit message: '
Parts:
- added J7: Conn_01x02, Connector_PinHeader_2.54mm:PinHeader_1x02_P2.54mm_Vertical, F.Cu at (38.1, 19.6)
Routing:
- net AGND: track 37.9 -> 51.9 mm, vias 14 -> 23
- net +5V: track 10.3 -> 18.6 mm

Commit message: minor changes in stiffener layers
Other:
- board text added: "Stiffener 1: Polyamide Stiffener 1 Thickness: 0.2mm Stiffener 1 Location: see User.1 layer"
- board text added: "Stiffener 2: FR4 Stiffener 2 Thickness: 0.2mm Stiffener 2 Location: see User.2 layer"
- board text removed: "camera"
Changed lines of the file:
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@@
 	)
 	(gr_rect
-		(start 59.622265 57.369144)
-		(end 68.122265 65.869144)
+		(start 18.960265 16.619144)
+		(end 104.684265 46.569144)
 		(stroke
-			(width 0.1)
-			(type default)
+			(width 0.2)
+			(type solid)
 		)
 		(fill no)
-		(layer "Dwgs.User")
+		(layer "Edge.Cuts")
 	)
 	(gr_line
@@
 			(type solid)
 		)
-		(layer "Dwgs.User")
+		(layer "User.1")
 	)
 	(gr_line
@@
 			(type solid)
 		)
-		(layer "Dwgs.User")
+		(layer "User.1")
 	)
-	(gr_rect
-		(start 76.622265 55.369144)
-		(end 80.922265 67.869144)
+	(gr_line
+		(start 82.022265 17.019144)
+		(end 85.022265 23.019144)
 		(stroke
 			(width 0.1)
-			(type default)
+			(type solid)
 		)
-		(fill no)
-		(layer "Dwgs.User")
+		(layer "User.1")
 	)
 	(gr_line
-		(start 82.022265 18.719144)
-		(end 85.022265 23.019144)
+		(start 85.022265 41.019144)
+		(end 82.022265 46.319144)
 		(stroke
 			(width 0.1)
-			(type default)
+			(type solid)
 		)
-		(layer "Dwgs.User")
+		(layer "User.1")
 	)
-	(gr_rect
-		(start 68.122265 58.369144)
-		(end 76.622265 64.869144)
+	(gr_line
+		(start 53.022265 23.019144)
+		(end 56.022265 17.019144)
 		(stroke
 			(width 0.1)
-			(type default)
+			(type solid)
 		)
-		(fill no)
-		(layer "Dwgs.User")
+		(layer "User.1")
 	)
 	(gr_line
-		(start 85.022265 41.019144)
-		(end 82.022265 45.019144)
+		(start 56.022265 17.019144)
+		(end 82.022265 17.019144)
 		(stroke
 			(width 0.1)
-			(type default)
+			(type solid)
 		)
-		(layer "Dwgs.User")
+		(layer "User.1")
 	)
-	(gr_rect
-		(start 31.522265 17.519144)
-		(end 46.522265 22.519144)
+	(gr_line
+		(start 56.022265 46.319144)
+		(end 53.022265 41.019144)
 		(stroke
 			(width 0.1)
 			(type solid)
 		)
-		(fill no)
-		(layer "Dwgs.User")
+		(layer "User.1")
 	)
 	(gr_line
-		(start 53.022265 23.019144)
-		(end 56.022265 18.719144)
+		(start 82.022265 46.319144)
+		(end 56.022265 46.319144)
 		(stroke
 			(width 0.1)
-			(type default)
+			(type solid)
 		)
-		(layer "Dwgs.User")
+		(layer "User.1")
 	)
-	(gr_line
-		(start 56.022265 18.719144)
-		(end 82.022265 18.719144)
+	(gr_rect
+		(start 54.172265 25.819144)
+		(end 62.672265 34.319144)
 		(stroke
 			(width 0.1)
 			(type solid)
 		)
-		(layer "Dwgs.User")
+		(fill no)
+		(layer "User.2")
 	)
-	(gr_line
-		(start 56.022265 45.019144)
-		(end 53.022265 41.019144)
+	(gr_rect
+		(start 71.172265 23.819144)
+		(end 75.472265 36.319144)
 		(stroke
 			(width 0.1)
-			(type default)
+			(type solid)
 		)
-		(layer "Dwgs.User")
+		(fill no)
+		(layer "User.2")
 	)
-	(gr_line
-		(start 82.022265 45.019144)
-		(end 56.022265 45.019144)
+	(gr_rect
+		(start 62.672265 26.819144)
+		(end 71.172265 33.319144)
 		(stroke
 			(width 0.1)
 			(type solid)
 		)
-		(layer "Dwgs.User")
+		(fill no)
+		(layer "User.2")
 	)
 	(gr_rect
-		(start 18.960265 16.619144)
-		(end 104.684265 46.569144)
+		(start 31.522265 17.519144)
+		(end 46.522265 22.519144)
 		(stroke
-			(width 0.2)
+			(width 0.1)
 			(type solid)
 		)
 		(fill no)
-		(layer "Edge.Cuts")
+		(layer "User.2")
 	)
 	(gr_text "VDD"
@@
 		)
 	)
-	(gr_text "camera"
-		(at 61.012265 62.119144 0)
-		(layer "Dwgs.User")
+	(gr_text "Stiffener 1: Polyamide\nStiffener 1 Thickness: 0.2mm\nStiffener 1 Location: see User.1 layer"
+		(at 68.422265 56.269144 0)
+		(layer "User.3")
+		(effects
+			(font
+				(size 1 1)
+				(thickness 0.15)
+			)
+			(justify left bottom)
+		)
+	)
+	(gr_text "Stiffener 2: FR4\nStiffener 2 Thickness: 0.2mm\nStiffener 2 Location: see User.2 layer"
+		(at 68.472265 62.369144 0)
+		(layer "User.3")
 		(effects
 			(font
@@
 	)
 	(group ""
-		(members "f1678b0e-b19c-46ce-8f6d-c3e9ffc45a36")
-	)
-	(group ""
-		(members "2a52d574-0656-4e15-8bfe-fbb119ecb65f" "5111bb17-f799-4b58-9334-4d2f49095859"
-			"677b45ac-e662-49c3-994c-a141554a7526" "e3884ea3-72cc-4dbe-99af-4d2f5ed05d94"
+		(members "1ebd8789-4a47-4d09-9c4b-4094bd325f70" "36762440-41da-4131-bd75-e7dcc13ee28b"
+			"ac4c3cb7-98fb-4352-97f0-7531626d58a9"
 		)
 	)

Commit message: change default clearance, add fabrication files
Routing:
- net AGND: track 51.9 -> 47.3 mm, vias 23 -> 22
- net +3.3V: track 160.4 -> 161.3 mm
Other:
- board size 85.7 x 30 mm -> 85.7 x 31.1 mm
Changed lines of the file:
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@@
 		(grid_origin 19.022265 47.519144)
 		(pcbplotparams
-			(layerselection 0x00000000_00000000_55555555_5755f5ff)
+			(layerselection 0x00000000_00000000_555557d5_5755f5af)
 			(plot_on_all_layers_selection 0x00000000_00000000_00000000_00000000)
 			(disableapertmacros no)
@@
 			(outputformat 1)
 			(mirror no)
-			(drillshape 1)
+			(drillshape 0)
 			(scaleselection 1)
-			(outputdirectory "")
+			(outputdirectory "fab_files/gerber/")
 		)
 	)
@@
 	)
 	(gr_rect
-		(start 18.960265 16.619144)
-		(end 104.684265 46.569144)
+		(start 18.960265 15.919144)
+		(end 104.684265 47.019144)
 		(stroke
 			(width 0.2)
@@
 	)
 	(segment
+		(start 63.4625 27.5125)
+		(end 63.915621 27.5125)
+		(width 0.2)
+		(layer "F.Cu")
+		(net 1)
+	)
+	(segment
 		(start 69.7 34.446879)
 		(end 70.193434 34.940313)
@@
 	)
 	(segment
+		(start 63.915621 27.5125)
+		(end 64.242265 27.839144)
+		(width 0.2)
+		(layer "F.Cu")
+		(net 1)
+	)
+	(segment
 		(start 64.215621 31.5125)
 		(end 64.222265 31.519144)
@@
 	)
 	(segment
-		(start 66.9 34.24992)
+		(start 66.9 34.705276)
 		(end 66.9 33.75)
 		(width 0.15)
@@
 	)
 	(segment
-		(start 68.572265 22.019144)
-		(end 68.572265 21.317144)
-		(width 0.5)
+		(start 66.572265 34.891409)
+		(end 66.713867 34.891409)
+		(width 0.15)
 		(layer "F.Cu")
 		(net 3)
@@
 	)
 	(segment
-		(start 72.046292 29.7125)
-		(end 72.222265 29.888472)
-		(width 0.2)
+		(start 68.572265 22.019144)
+		(end 68.572265 20.969144)
+		(width 0.4)
 		(layer "F.Cu")
 		(net 3)
 	)
 	(segment
-		(start 68.572265 21.317144)
-		(end 69.920265 19.969144)
-		(width 0.5)
+		(start 72.046292 29.7125)
+		(end 72.222265 29.888472)
+		(width 0.2)
 		(layer "F.Cu")
 		(net 3)
@@
 	)
 	(segment
+		(start 68.572265 20.969144)
+		(end 68.823765 20.717644)
+		(width 0.4)
+		(layer "F.Cu")
+		(net 3)
+	)
+	(segment
+		(start 66.713867 34.891409)
+		(end 66.9 34.705276)
+		(width 0.15)
+		(layer "F.Cu")
+		(net 3)
+	)
+	(segment
 		(start 68.512267 23.769144)
 		(end 68.792265 23.769144)
@@
 	)
 	(segment
-		(start 69.920265 19.969144)
-		(end 72.272265 19.969144)
-		(width 0.5)
-		(layer "F.Cu")
-		(net 3)
-	)
-	(segment
-		(start 66.572265 34.577655)
-		(end 66.9 34.24992)
-		(width 0.15)
-		(layer "F.Cu")
-		(net 3)
-	)
-	(segment
-		(start 66.572265 34.891409)
-		(end 66.572265 34.577655)
-		(width 0.15)
+		(start 61.982265 26.769144)
+		(end 61.982265 26.159144)
+		(width 0.2)
 		(layer "F.Cu")
 		(net 3)
 	)
 	(segment
-		(start 61.982265 26.769144)
-		(end 61.982265 26.159144)
-		(width 0.2)
+		(start 69.733265 20.365586)
+		(end 69.733265 20.156144)
+		(width 0.4)
 		(layer "F.Cu")
 		(net 3)
@@
 	)
 	(segment
+		(start 69.920265 19.969144)
+		(end 72.272265 19.969144)
+		(width 0.4)
+		(layer "F.Cu")
+		(net 3)
+	)
+	(segment
 		(start 68.1 24.181411)
 		(end 68.1 26.875)
@@
 	)
 	(segment
-		(start 66.651 37.105407)
-		(end 67.222265 37.676672)
-		(width 0.5)
+		(start 66.586132 34.905276)
+		(end 66.572265 34.891409)
+		(width 0.15)
 		(layer "F.Cu")
 		(net 3)
@@
 	)
 	(segment
+		(start 66.651 37.105407)
+		(end 67.222265 37.676672)
+		(width 0.5)
+		(layer "F.Cu")
+		(net 3)
+	)
+	(segment
 		(start 66.7 34.919144)
 		(end 66.8 35.019144)
@@
 	)
 	(segment
-		(start 66.586132 34.905276)
-		(end 66.572265 34.891409)
-		(width 0.15)
+		(start 69.381207 20.717644)
+		(end 69.733265 20.365586)
+		(width 0.4)
+		(layer "F.Cu")
+		(net 3)
+	)
+	(segment
+		(start 68.823765 20.717644)
+		(end 69.381207 20.717644)
+		(width 0.4)
+		(layer "F.Cu")
+		(net 3)
+	)
+	(segment
+		(start 69.733265 20.156144)
+		(end 69.920265 19.969144)
+		(width 0.4)
 		(layer "F.Cu")
 		(net 3)
@@
 	)
 	(segment
-		(start 41.822265 20.769144)
-		(end 41.822265 23.669144)
-		(width 0.5)
-		(layer "F.Cu")
-		(net 4)
-	)
-	(segment
 		(start 75.402265 29.319144)
 		(end 75.402265 28.319144)
@@
 	)
 	(segment
-		(start 40.622265 19.569144)
-		(end 41.822265 20.769144)
-		(width 0.5)
-		(layer "F.Cu")
-		(net 4)
-	)
-	(segment
 		(start 75.422265 43.069144)
 		(end 74.872265 43.069144)
@@
 		(layers "F.Cu" "B.Cu")
 		(net 4)
-	)
-	(via
-		(at 41.822265 23.669144)
-		(size 0.6)
-		(drill 0.3)
-		(layers "F.Cu" "B.Cu")
-		(net 4)
