File: Connector_board/Connector_board.kicad_pcb (KiCad board)
At the start: 2 copper layers, 54.2 x 20 mm, 6 parts, among them J1 USB_B_Micro, J2 Conn_02x04_Counter_Clockwise, J3 Conn_02x06_Counter_Clockwise, J4 Conn_02x07_Counter_Clockwise

Commit message: layout finalized (?)
Parts:
- added J5: SM03B-SRSS-TB, Connector_JST:JST_SH_SM03B-SRSS-TB_1x03-1MP_P1.00mm_Horizontal, F.Cu at (26.7, 36.0)
- moved D1 3.76 mm to (28.9, 40.9), turned to 180 degrees
Connections:
- J2 pad 5: GND -> /SWCLK_1
- J2 pad 7: unconnected-(J2-Pin_7-Pad7) -> /SWD_1
- J2 pad 8: unconnected-(J2-Pin_8-Pad8) -> GND
Routing:
- net /SWCLK_1: track 0.00 -> 11.7 mm
- net /SWD_1: track 0.00 -> 9.29 mm

Commit message: connector board updated
Parts:
- moved J4 1.05 mm to (67.3, 42.1)
Connections:
- J3 pad 11: /IMAGE_OUT_1_1- -> /POSITION_OUT_1
- J3 pad 7: /POSITION_OUT_1 -> /IMAGE_OUT_2_1-
- J3 pad 9: /IMAGE_OUT_2_1- -> /IMAGE_OUT_1_1-
- J4 pad 5: /POSITION_OUT_1 -> /IMAGE_OUT_2_1-
- J4 pad 7: /IMAGE_OUT_2_1- -> /IMAGE_OUT_1_1-
- J4 pad 9: /IMAGE_OUT_1_1- -> /POSITION_OUT_1
Routing:
- net /POSITION_OUT_1: track 17.7 -> 19.9 mm
Changed lines of the file:
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@@
 	(footprint "Connector_Molex:Molex_SlimStack_502430-1410_2x07_P0.40mm_Vertical"
 		(layer "F.Cu")
-		(at 67.295 41.05 90)
+		(at 67.255 42.1 90)
 		(descr "Molex SlimStack Fine-Pitch SMT Board-to-Board Connectors, 502430-1410, 14 Pins (http://www.molex.com/pdm_docs/sd/5024301410_sd.pdf), generated with kicad-footprint-generator")
 		(tags "connector Molex SlimStack vertical")
@@
 			(size 0.22 0.66)
 			(layers "F.Cu" "F.Mask" "F.Paste")
-			(net 16 "/POSITION_OUT_1")
+			(net 14 "/IMAGE_OUT_2_1-")
 			(pinfunction "Pin_5")
 			(pintype "passive")
@@
 			(size 0.22 0.66)
 			(layers "F.Cu" "F.Mask" "F.Paste")
-			(net 14 "/IMAGE_OUT_2_1-")
+			(net 9 "/IMAGE_OUT_1_1-")
 			(pinfunction "Pin_7")
 			(pintype "passive")
@@
 			(size 0.22 0.66)
 			(layers "F.Cu" "F.Mask" "F.Paste")
-			(net 9 "/IMAGE_OUT_1_1-")
+			(net 16 "/POSITION_OUT_1")
 			(pinfunction "Pin_9")
 			(pintype "passive")
@@
 			(layers "*.Cu" "*.Mask")
 			(remove_unused_layers no)
-			(net 16 "/POSITION_OUT_1")
+			(net 14 "/IMAGE_OUT_2_1-")
 			(pinfunction "Pin_7")
 			(pintype "passive")
@@
 			(layers "*.Cu" "*.Mask")
 			(remove_unused_layers no)
-			(net 14 "/IMAGE_OUT_2_1-")
+			(net 9 "/IMAGE_OUT_1_1-")
 			(pinfunction "Pin_9")
 			(pintype "passive")
@@
 			(layers "*.Cu" "*.Mask")
 			(remove_unused_layers no)
-			(net 9 "/IMAGE_OUT_1_1-")
+			(net 16 "/POSITION_OUT_1")
 			(pinfunction "Pin_11")
 			(pintype "passive")
@@
 	)
 	(gr_text "IO1-"
-		(at 50.65 37 0)
+		(at 50.8 39.5 0)
 		(layer "F.SilkS")
 		(effects
@@
 	)
 	(gr_text "PO"
-		(at 50.65 42.1 0)
+		(at 50.8 37 0)
 		(layer "F.SilkS")
 		(effects
@@
 	)
 	(gr_text "IO2-"
-		(at 50.65 39.45 0)
+		(at 50.75 42 0)
 		(layer "F.SilkS")
 		(effects
@@
 	)
 	(segment
-		(start 51.525 39.15)
-		(end 63.9 39.15)
+		(start 50.99 38.89)
+		(end 54.1 42)
 		(width 0.2)
 		(layer "F.Cu")
@@
 	)
 	(segment
-		(start 48.725 36.35)
-		(end 51.525 39.15)
+		(start 65.15 42)
+		(end 65.25 42.1)
 		(width 0.2)
 		(layer "F.Cu")
@@
 	)
 	(segment
-		(start 63.9 39.15)
-		(end 65.4 40.65)
+		(start 48.725 38.89)
+		(end 50.99 38.89)
 		(width 0.2)
 		(layer "F.Cu")
@@
 	)
 	(segment
-		(start 65.4 40.65)
-		(end 66.44 40.65)
+		(start 65.25 42.1)
+		(end 66.4 42.1)
 		(width 0.2)
 		(layer "F.Cu")
@@
 	)
 	(segment
-		(start 64.75 41.85)
-		(end 66.44 41.85)
+		(start 54.1 42)
+		(end 65.15 42)
+		(width 0.2)
+		(layer "F.Cu")
+		(net 9)
+	)
+	(segment
+		(start 52.7 42.9)
+		(end 66.4 42.9)
 		(width 0.2)
 		(layer "F.Cu")
@@
 	)
 	(segment
+		(start 51.63 43.97)
+		(end 52.7 42.9)
+		(width 0.2)
+		(layer "F.Cu")
+		(net 10)
+	)
+	(segment
 		(start 48.725 43.97)
-		(end 50.195 42.5)
+		(end 51.63 43.97)
 		(width 0.2)
 		(layer "F.Cu")
@@
 	)
 	(segment
-		(start 64.1 42.5)
-		(end 64.75 41.85)
-		(width 0.2)
-		(layer "F.Cu")
-		(net 10)
-	)
-	(segment
-		(start 50.195 42.5)
-		(end 64.1 42.5)
-		(width 0.2)
-		(layer "F.Cu")
-		(net 10)
-	)
-	(segment
-		(start 51.535 43.7)
-		(end 64 43.7)
+		(start 54.15 43.3)
+		(end 66.4 43.3)
 		(width 0.2)
 		(layer "F.Cu")
@@
 	)
 	(segment
-		(start 64 43.7)
-		(end 65.45 42.25)
+		(start 50.94 46.51)
+		(end 54.15 43.3)
 		(width 0.2)
 		(layer "F.Cu")
@@
 	(segment
 		(start 48.725 46.51)
-		(end 51.535 43.7)
+		(end 50.94 46.51)
 		(width 0.2)
 		(layer "F.Cu")
@@
 	)
 	(segment
-		(start 65.45 42.25)
-		(end 66.44 42.25)
-		(width 0.2)
-		(layer "F.Cu")
-		(net 11)
-	)
-	(segment
-		(start 48.725 38.89)
-		(end 50.235 40.4)
+		(start 48.725 41.43)
+		(end 51.63 41.43)
 		(width 0.2)
 		(layer "F.Cu")
@@
 	)
 	(segment
-		(start 64.05 40.4)
-		(end 64.7 41.05)
-		(width 0.2)
-		(layer "F.Cu")
-		(net 14)
-	)
-	(segment
-		(start 50.235 40.4)
-		(end 64.05 40.4)
-		(width 0.2)
-		(layer "F.Cu")
-		(net 14)
-	)
-	(segment
-		(start 64.7 41.05)
-		(end 66.44 41.05)
+		(start 51.63 41.43)
+		(end 52.7 42.5)
 		(width 0.2)
 		(layer "F.Cu")
@@
 		(width 0.2)
 		(layer "F.Cu")
+		(net 14)
+	)
+	(segment
+		(start 52.7 42.5)
+		(end 66.4 42.5)
+		(width 0.2)
+		(layer "F.Cu")
+		(net 14)
+	)
+	(segment
+		(start 55.999 41.599)
+		(end 65.399 41.599)
+		(width 0.2)
+		(layer "F.Cu")
 		(net 16)
 	)
 	(segment
-		(start 66.44 41.45)
-		(end 48.745 41.45)
-		(width 0.2)
-		(layer "F.Cu")
+		(start 65.399 41.599)
+		(end 65.5 41.7)
+		(width 0.2)
+		(layer "F.Cu")
+		(net 16)
+	)
+	(segment
+		(start 48.725 36.35)
+		(end 50.75 36.35)
+		(width 0.2)
+		(layer "F.Cu")
+		(net 16)
+	)
+	(segment
+		(start 50.75 36.35)
+		(end 55.999 41.599)
+		(width 0.2)
+		(layer "F.Cu")
+		(net 16)
+	)
+	(segment
+		(start 65.5 41.7)
+		(end 66.4 41.7)
+		(width 0.2)
+		(layer "F.Cu")

Commit message: '
Parts:
- J2, J4: moved to B.Cu
- moved J4 3.30 mm to (64.0, 42.0)
- moved J2 0.34 mm to (35.1, 42.6)
Routing:
- net /USB_D1-: track 12.8 -> 17.4 mm, vias 0 -> 1
- net /USB_D1+: track 12.8 -> 17.3 mm, vias 0 -> 1
- net /SWCLK_1: track 11.7 -> 15.6 mm, vias 0 -> 1
- net /IMAGE_OUT_2_1-: track 18.1 -> 20.7 mm, vias 0 -> 1
- net /IMAGE_OUT_2_1+: track 18.1 -> 20.5 mm, vias 0 -> 1
- net /SWD_1: track 9.29 -> 11.3 mm, vias 0 -> 1
- net /IMAGE_OUT_1_1+: track 19.0 -> 19.9 mm, vias 0 -> 1
- net /IMAGE_OUT_1_1-: track 19.0 -> 19.9 mm, vias 0 -> 1
- net /POSITION_OUT_1: track 19.9 -> 20.8 mm, vias 0 -> 1
