File: Connector_board/Connector_board.kicad_sch (KiCad schematic)
At the start: 6 parts, among them J1 USB_B_Micro, J2 Conn_02x04_Counter_Clockwise, J3 Conn_02x06_Counter_Clockwise, J4 Conn_02x07_Counter_Clockwise

Commit message: layout finalized (?)
Parts:
- added J5: SM03B-SRSS-TB, Connector_JST:JST_SH_SM03B-SRSS-TB_1x03-1MP_P1.00mm_Horizontal, symbol Connector_Generic_MountingPin:Conn_01x03_MountingPin
Connections:
- net GND: now also J2.8 (Pin_8), J5.2 (Pin_2), J5.MP (MountPin); no longer J2.5 (Pin_5)
- net SWD_1: now reaches J2.7 (Pin_7)
- net SWD_1: now also J5.1 (Pin_1)
- new net SWCLK_1: J2.5 (Pin_5), J5.3 (Pin_3)
- no-connect marks 19 -> 17
Other:
- note added: "JST Debug Connector"
- moved on the sheet: J1, J2

Commit message: connector board updated
Connections:
- net IMAGE_OUT_1_1-: now also J3.9 (Pin_9), J4.7 (Pin_7); no longer J3.11 (Pin_11), J4.9 (Pin_9)
- net IMAGE_OUT_2_1-: now also J3.7 (Pin_7), J4.5 (Pin_5); no longer J3.9 (Pin_9), J4.7 (Pin_7)
- net POSITION_OUT_1: now also J3.11 (Pin_11), J4.9 (Pin_9); no longer J3.7 (Pin_7), J4.5 (Pin_5)
Changed lines of the file:
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@@
 	)
 	(label "IMAGE_OUT_1_1-"
-		(at 36.83 83.82 180)
+		(at 36.83 81.28 180)
+		(effects
+			(font
+				(size 1.27 1.27)
+			)
+			(justify right bottom)
+		)
+	)
+	(label "IMAGE_OUT_1_1-"
+		(at 80.01 78.74 180)
 		(effects
 			(font
@@
 		)
 	)
-	(label "IMAGE_OUT_1_1-"
-		(at 80.01 81.28 180)
+	(label "USB_D1-"
+		(at 63.5 31.75 180)
 		(effects
 			(font
@@
 		)
 	)
-	(label "USB_D1-"
-		(at 63.5 31.75 180)
+	(label "POSITION_OUT_1"
+		(at 80.01 81.28 180)
 		(effects
 			(font
@@
 	)
 	(label "IMAGE_OUT_2_1-"
-		(at 80.01 78.74 180)
-		(effects
-			(font
-				(size 1.27 1.27)
-			)
-			(justify right bottom)
-		)
-	)
-	(label "POSITION_OUT_1"
 		(at 36.83 78.74 180)
 		(effects
@@
 		)
 	)
-	(label "IMAGE_OUT_2_1+"
-		(at 36.83 76.2 180)
+	(label "IMAGE_OUT_2_1-"
+		(at 80.01 76.2 180)
 		(effects
 			(font
@@
 		)
 	)
-	(label "POSITION_OUT_1"
-		(at 80.01 76.2 180)
+	(label "IMAGE_OUT_2_1+"
+		(at 36.83 76.2 180)
 		(effects
 			(font
@@
 		)
 	)
-	(label "IMAGE_OUT_2_1-"
-		(at 36.83 81.28 180)
+	(label "POSITION_OUT_1"
+		(at 36.83 83.82 180)
 		(effects
 			(font

Commit message: test PCB version 2 completed
Parts:
- removed J2: Conn_02x04_Counter_Clockwise, Connector_Molex:Molex_SlimStack_502430-0820_2x04_P0.40mm_Vertical, symbol Connector_Generic:Conn_02x04_Odd_Even
- removed J3: Conn_02x06_Counter_Clockwise, Connector_PinHeader_2.54mm:PinHeader_2x06_P2.54mm_Vertical, symbol Connector_Generic:Conn_02x06_Odd_Even
- added J3: Conn_02x07_Counter_Clockwise, Connector_Molex:Molex_SlimStack_502430-1410_2x07_P0.40mm_Vertical, symbol Connector_Generic:Conn_02x07_Odd_Even
- added J4: Conn_02x07_Odd_Even, Connector_PinHeader_2.54mm:PinHeader_2x07_P2.54mm_Vertical, symbol Connector_Generic:Conn_02x07_Odd_Even
- renumbered J5 to J1, J1 to J2, J4 to J5
Connections:
- net IMAGE_OUT_2_1+ is gone; now on net POSITION_OUT_1: J5.3 (Pin_3)
- net GND: now also J5.14 (Pin_14), J3.14 (Pin_14), J4.2 (Pin_2); no longer J5.11 (Pin_11)
- net POSITION_OUT_1: now also J4.11 (Pin_11); no longer J5.9 (Pin_9)
- net SWCLK_1: now also J3.3 (Pin_3)
- net SWD_1: now also J3.1 (Pin_1)
- net USB_D1+: now also J3.7 (Pin_7)
- net USB_D1-: now also J3.5 (Pin_5)
- net FPGA_EN: now reaches J5.13 (Pin_13)
- net FPGA_EN: now also J4.1 (Pin_1)
- net IMAGE_CLK: now reaches J5.4 (Pin_4)
- net IMAGE_CLK: now also J4.12 (Pin_12)
- net VSYNC_OUT: now reaches J5.6 (Pin_6)
- net VSYNC_OUT: now also J4.10 (Pin_10)
- net POSITION_OUT_CLK: now reaches J5.8 (Pin_8)
- net POSITION_OUT_CLK: now also J4.8 (Pin_8)
- net +3V3 renamed +5V
- net +5V: now also J3.2 (Pin_2)
- net IMAGE_OUT_1_1+ renamed HREF_OUT
- net HREF_OUT: now also J4.13 (Pin_13)
- net IMAGE_OUT_1_1- renamed IMAGE_OUT_3
- net IMAGE_OUT_3: now also J4.7 (Pin_7)
- net IMAGE_OUT_2_1- renamed IMAGE_OUT_4
- net IMAGE_OUT_4: now also J4.9 (Pin_9)
- new net IMAGE_OUT_1: J4.3 (Pin_3), J5.11 (Pin_11)
- new net IMAGE_OUT_2: J4.5 (Pin_5), J5.9 (Pin_9)
- no-connect marks 17 -> 14
Other:
- moved on the sheet: J5

Commit message: refined 5V net isolation
Connections:
- net +5V: no longer J3.2 (Pin_2)
- no-connect marks 14 -> 15
Changed lines of the file:
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@@
+	)
+	(no_connect
+		(at 76.2 25.4)
 	)
 	(no_connect
@@
 					(unit 1)
 				)
-			)
-		)
-	)
-	(symbol
-		(lib_id "power:+5V")
-		(at 76.2 25.4 0)
-		(unit 1)
-		(body_style 1)
-		(exclude_from_sim no)
-		(in_bom yes)
-		(on_board yes)
-		(in_pos_files yes)
-		(dnp no)
-		(property "Reference" "#PWR04"
-			(at 76.2 29.21 0)
-			(hide yes)
-			(show_name no)
-			(do_not_autoplace no)
-			(effects
-				(font
-					(size 1.27 1.27)
-				)
-			)
-		)
-		(property "Value" "+5V"
-			(at 78.232 22.352 0)
-			(show_name no)
-			(do_not_autoplace no)
-			(effects
-				(font
-					(size 1.27 1.27)
-				)
-			)
-		)
-		(property "Footprint" ""
-			(at 76.2 25.4 0)
-			(hide yes)
-			(show_name no)
-			(do_not_autoplace no)
-			(effects
-				(font
-					(size 1.27 1.27)
-				)
-			)
-		)
-		(property "Datasheet" ""
-			(at 76.2 25.4 0)
-			(hide yes)
-			(show_name no)
-			(do_not_autoplace no)
-			(effects
-				(font
-					(size 1.27 1.27)
-				)
-			)
-		)
-		(property "Description" "Power symbol creates a global label with name \"+5V\""
-			(at 76.2 25.4 0)
-			(hide yes)
-			(show_name no)
-			(do_not_autoplace no)
-			(effects
-				(font
-					(size 1.27 1.27)
-				)
-			)
-		)
-		(pin "1"
-		)
-		(instances
-			(project "Connector_board"
-				(path "/d47a3cbb-9124-4e72-898a-608406011dc9"
-					(reference "#PWR04")
-					(unit 1)
-				)
